File: KiCad Dir/TKD_DBTypeC_r1.kicad_pcb (KiCad board)
At the start: 2 copper layers, 8 parts, among them J1 JST-SH-SM04B-SRSS-TB

Commit message: pcb/schemea update
Parts:
- added H1: MountingHole, MountingHole:MountingHole_2.7mm_M2.5_DIN965_Pad, F.Cu at (57.5, 75.0)
- added H2: MountingHole, MountingHole:MountingHole_2.7mm_M2.5_DIN965_Pad, F.Cu at (55.0, 60.0)
- added H3: MountingHole, MountingHole:MountingHole_2.7mm_M2.5_DIN965_Pad, F.Cu at (75.0, 75.0)
- added H4: MountingHole_Pad, MountingHole:MountingHole_2.7mm_M2.5_DIN965_Pad, F.Cu at (77.5, 60.0)
- moved D1 26.5 mm to (66.3, 64.3)
- moved F1 26.5 mm to (72.3, 64.2)
- moved FB2 26.5 mm to (62.4, 65.6)
- moved J1 26.5 mm to (66.4, 71.1)
- moved R1 26.5 mm to (72.3, 60.7)
- moved R2 26.5 mm to (59.6, 60.7)
- moved USB1 26.5 mm to (68.9, 61.3)
- moved FB1 26.5 mm to (62.4, 63.5)

Commit message: Edge cuts placed, r1 done
Parts:
- moved H1 2.84 mm to (59.7, 73.2)
- moved H3 2.62 mm to (73.1, 73.2)
- moved H2 2.51 mm to (53.8, 57.8)
- moved H4 2.31 mm to (78.2, 57.8)
Routing:
- net GND: track 6.90 -> 46.7 mm, vias 0 -> 2
- net VBUS: track 9.87 -> 15.5 mm
- net +5V: track 5.59 -> 5.07 mm
- added copper zone on B.Cu, net GND
- added copper zone on F.Cu, net GND
Other:
- board outline added: 30 x 21.5 mm
- net class POWER added: clearance 0.2, trace_width 0.5, via_dia 1, via_drill 0.6
- board text added: "TKDB-TypeC R1.0"
